Commit message: Fix mate-limit/axis/color/origin bugs, add root_mate_name, fold xacro export into package
Fixes an "explosion" featureType crash that silently discarded mate
limits for entire assemblies, corrects the revolute joint axis sign
and limit convention, makes link color a configurable uniform default,
and snaps floating-point origin noise to zero. Adds root_mate_name to
KinematicGraph.from_cad() so the kinematic root can be selected via a
named mate-to-origin instead of a throwaway dummy fixed part.

Also moves xacro_export.py's URDF-to-xacro conversion into the package
as onshape_robotics_toolkit.formats.xacro, and documents how to consume
this fork as a git dependency from another repo.

Co-Authored-By: Claude Sonnet 5 <noreply@anthropic.com>

File: tests/data/assembly_expected.urdf (robot description, URDF)
Before this commit: robot test_robot, 9 links, 8 joints
Joints:
- joint Revolute_1: axis 0 0 -1 -> 0 0 1
- joint Revolute_1-1: axis 0 0 -1 -> 0 0 1
- joint Revolute_1-2: axis 0 0 -1 -> 0 0 1
- joint Revolute_1-3: axis 0 0 -1 -> 0 0 1
- joint Revolute_2: axis 0 0 -1 -> 0 0 1
- joint Revolute_2-1: axis 0 0 -1 -> 0 0 1
- joint Revolute_3: axis 0 0 -1 -> 0 0 1
- joint Revolute_3-1: axis 0 0 -1 -> 0 0 1
